Commit message: Robot moves and does not flip over. Note that the robot does not move up ramps

File: robots/goat.urdf.xacro (robot description, xacro)
@@ -11,5 +11,5 @@
     <link name="base_link">
         <inertial>
-            <origin xyz="0 0 0.5" rpy="0 0 0"/>
+            <origin xyz="0 0 -0.2" rpy="0 0 0"/>
             <mass value="10"/>
             <inertia ixx="0.1"  ixy="0"  ixz="0" iyy="0.1" iyz="0" izz="0.1" />
